File: KiCAD/Tiny486.kicad_sch (KiCad schematic)
At the start: 0 parts

Commit message: Begin schematic work
Parts:
- added C? (x2): 10u, symbol Device:C_Small
- added C? (x2): 0.1u, symbol Device:C_Small
- added C? (x2): 1u, symbol Device:C_Small
- added R? (x2): 0, symbol Device:R_Small
- added U?: SC410-100, 486Parts:SC410_BGA292, symbol 486Parts:SC410-100
Connections:
- new net: U?.M3 (RESERVED), U?.N2 (RESERVED), U?.P1 (RESERVED), U?.P3 (RESERVED), U?.R2 (RESERVED), U?.R3 (RESERVED), U?.T2 (RESERVED), U?.U1 (RESERVED), U?.V1 (RESERVED), U?.W5 (RESERVED)
- new net +3V3: R?.1, R?.1
- new net D0: U?.B10 (D0)
- new net D1: U?.A10 (D1)
- new net D10: U?.C7 (D10)
- new net D11: U?.B6 (D11)
- new net D12: U?.A5 (D12)
- new net D13: U?.C6 (D13)
- new net D14: U?.B5 (D14)
- new net D15: U?.A4 (D15)
- new net D2: U?.C9 (D2)
- new net D3: U?.B9 (D3)
- new net D4: U?.A9 (D4)
- new net D5: U?.B8 (D5)
- new net D6: U?.C8 (D6)
- new net D7: U?.A7 (D7)
- new net D8: U?.B7 (D8)
- new net D9: U?.A6 (D9)
- new net GND: C?.2, C?.2, C?.2, C?.2, C?.2, C?.2, U?.D10 (GND), U?.D11 (GND), U?.D12 (GND), U?.D4 (GND), U?.D5 (GND), U?.D6 (GND), U?.D7 (GND), U?.D8 (GND), U?.D9 (GND), U?.E4 (GND), U?.F4 (GND), U?.G4 (GND), U?.H10 (GND), U?.H11 (GND), U?.H12 (GND), U?.H13 (GND), U?.H4 (GND), U?.H8 (GND), U?.H9 (GND), U?.J10 (GND), U?.J11 (GND), U?.J12 (GND), U?.J13 (GND), U?.J4 (GND), U?.J8 (GND), U?.J9 (GND), U?.K10 (GND), U?.K11 (GND), U?.K12 (GND), U?.K13 (GND), U?.K8 (GND), U?.K9 (GND), U?.L10 (GND), U?.L11 (GND), U?.L12 (GND), U?.L13 (GND), U?.L8 (GND), U?.L9 (GND), U?.M10 (GND), U?.M11 (GND), U?.M12 (GND), U?.M13 (GND), U?.M8 (GND), U?.M9 (GND), U?.N10 (GND), U?.N11 (GND), U?.N12 (GND), U?.N13 (GND), U?.N8 (GND), U?.N9 (GND), U?.R17 (GND), U?.T17 (GND), U?.U10 (GND), U?.U11 (GND), U?.U12 (GND), U?.U13 (GND), U?.U14 (GND), U?.U15 (GND), U?.U16 (GND), U?.U17 (GND), U?.U5 (GND), U?.U6 (GND), U?.U7 (GND), U?.U8 (GND), U?.U9 (GND)
- new net SD0: U?.G3 (SD0/D16)
- new net SD1: U?.F2 (SD1/D17)
- new net SD10: U?.J1 (SD10/D26)
- new net SD11: U?.K1 (SD11/D27)
- new net SD12: U?.L1 (SD12/D28)
- new net SD13: U?.L2 (SD13/D29)
- new net SD14: U?.N1 (SD14/D30)
- new net SD15: U?.L3 (SD15/D31)
- new net SD2: U?.H3 (SD2/D18)
- new net SD3: U?.G2 (SD3/D19)
- new net SD4: U?.F1 (SD4/D20)
- new net SD5: U?.H2 (SD5/D21)
- new net SD6: U?.G1 (SD6/D22)
- new net SD7: U?.J2 (SD7/D23)
- new net SD8: U?.K3 (SD8/D24)
- new net SD9: U?.K2 (SD9/D25)
- new net VCC: C?.1, C?.1, C?.1, R?.2, U?.A13 (VCC), U?.A18 (VCC), U?.A8 (VCC), U?.B1 (VCC), U?.B16 (VCC), U?.B4 (VCC), U?.E1 (VCC), U?.E17 (VCC), U?.G17 (VCC), U?.H1 (VCC), U?.J17 (VCC), U?.J3 (VCC), U?.L17 (VCC), U?.M1 (VCC), U?.M17 (VCC), U?.M19 (VCC), U?.N17 (VCC), U?.P17 (VCC), U?.P18 (VCC), U?.T1 (VCC), U?.U18 (VCC), U?.V13 (VCC), U?.W9 (VCC), U?.Y1 (VCC), U?.Y16 (VCC)
- new net VCC_ANA: U?.W6 (VCC_A)
- new net VCC_CPU: C?.1, C?.1, C?.1, R?.2, U?.K4 (VCC_CPU), U?.L4 (VCC_CPU), U?.M4 (VCC_CPU), U?.N4 (VCC_CPU), U?.P4 (VCC_CPU), U?.R4 (VCC_CPU), U?.T4 (VCC_CPU)
- new net VCC_RTC: U?.W7 (VCC_RTC)
Other:
- note added: "CPU Power Rails"

Commit message: More schematic work
Parts:
- removed C? (x2): 10u, symbol Device:C_Small
- removed C? (x2): 0.1u, symbol Device:C_Small
- removed C? (x2): 1u, symbol Device:C_Small
- removed R? (x2): 0, symbol Device:R_Small
- removed U?: SC410-100, 486Parts:SC410_BGA292, symbol 486Parts:SC410-100
- added C1, C2, C7: 10u, symbol Device:C_Small
- added C10, C11, C12, C13, C14, C5, C6, C9: 0.1u, symbol Device:C_Small
- added C3, C4, C8: 1u, symbol Device:C_Small
- added R1, R2, R3: 0, symbol Device:R_Small
- added U1: SC410-100, 486Parts:SC410_BGA292, symbol 486Parts:SC410-100
- added U2: SST39VF040, symbol 486Parts:SST39VF040
- added U3: 74ALVC164245, Package_SO:TSSOP-48_6.1x12.5mm_P0.5mm, symbol 486Parts:74ALVC164245
- added U4, U5: K4E661612B, symbol 486Parts:K4E661612B
Connections:
- net +3V3: now also C1.1, C11.1, C13.1, C14.1, C3.1, C5.1, R1.1, R1.2, R2.1, R3.1, U1.A13 (VCC), U1.A18 (VCC), U1.A8 (VCC), U1.B1 (VCC), U1.B16 (VCC), U1.B4 (VCC), U1.E1 (VCC), U1.E17 (VCC), U1.G17 (VCC), U1.H1 (VCC), U1.J17 (VCC), U1.J3 (VCC), U1.L17 (VCC), U1.M1 (VCC), U1.M17 (VCC), U1.M19 (VCC), U1.N17 (VCC), U1.P17 (VCC), U1.P18 (VCC), U1.T1 (VCC), U1.U18 (VCC), U1.V13 (VCC), U1.W9 (VCC), U1.Y1 (VCC), U1.Y16 (VCC), U3.31 (VCCA), U3.42 (VCCA), U4.1 (VCC), U4.12 (VCC), U4.25 (VCC), U4.6 (VCC), U5.1 (VCC), U5.12 (VCC), U5.25 (VCC), U5.6 (VCC)
- net D0: now also U1.B10 (D0), U4.2 (D0)
- net D1: now also U1.A10 (D1), U4.3 (D1)
- net D10: now also U1.C7 (D10), U4.43 (D10)
- net D11: now also U1.B6 (D11), U4.44 (D11)
- net D12: now also U1.A5 (D12), U4.46 (D12)
- net D13: now also U1.C6 (D13), U4.47 (D13)
- net D14: now also U1.B5 (D14), U4.48 (D14)
- net D15: now also U1.A4 (D15), U4.49 (D15)
- net D2: now also U1.C9 (D2), U4.4 (D2)
- net D3: now also U1.B9 (D3), U4.5 (D3)
- net D4: now also U1.A9 (D4), U4.7 (D4)
- net D5: now also U1.B8 (D5), U4.8 (D5)
- net D6: now also U1.C8 (D6), U4.9 (D6)
- net D7: now also U1.A7 (D7), U4.10 (D7)
- net D8: now also U1.B7 (D8), U4.41 (D8)
- net D9: now also U1.A6 (D9), U4.42 (D9)
- net GND: now also C1.2, C10.2, C11.2, C12.2, C13.2, C14.2, C2.2, C3.2, C4.2, C5.2, C6.2, C7.2, C8.2, C9.2, U1.D10 (GND), U1.D11 (GND), U1.D12 (GND), U1.D4 (GND), U1.D5 (GND), U1.D6 (GND), U1.D7 (GND), U1.D8 (GND), U1.D9 (GND), U1.E4 (GND), U1.F4 (GND), U1.G4 (GND), U1.H10 (GND), U1.H11 (GND), U1.H12 (GND), U1.H13 (GND), U1.H4 (GND), U1.H8 (GND), U1.H9 (GND), U1.J10 (GND), U1.J11 (GND), U1.J12 (GND), U1.J13 (GND), U1.J4 (GND), U1.J8 (GND), U1.J9 (GND), U1.K10 (GND), U1.K11 (GND), U1.K12 (GND), U1.K13 (GND), U1.K8 (GND), U1.K9 (GND), U1.L10 (GND), U1.L11 (GND), U1.L12 (GND), U1.L13 (GND), U1.L8 (GND), U1.L9 (GND), U1.M10 (GND), U1.M11 (GND), U1.M12 (GND), U1.M13 (GND), U1.M8 (GND), U1.M9 (GND), U1.N10 (GND), U1.N11 (GND), U1.N12 (GND), U1.N13 (GND), U1.N8 (GND), U1.N9 (GND), U1.R17 (GND), U1.T17 (GND), U1.U10 (GND), U1.U11 (GND), U1.U12 (GND), U1.U13 (GND), U1.U14 (GND), U1.U15 (GND), U1.U16 (GND), U1.U17 (GND), U1.U5 (GND), U1.U6 (GND), U1.U7 (GND), U1.U8 (GND), U1.U9 (GND), U2.16 (GND), U3.10 (GND), U3.15 (GND), U3.21 (GND), U3.28 (GND), U3.34 (GND), U3.39 (GND), U3.4 (GND), U3.45 (GND), U4.26 (GND), U4.36 (OE), U4.39 (GND), U4.45 (GND), U4.50 (GND), U5.26 (GND), U5.36 (OE), U5.39 (GND), U5.45 (GND), U5.50 (GND)
- net SD0: now also U2.13 (D0), U3.2 (1B1)
- net SD1: now also U2.14 (D1), U3.3 (1B2)
- net SD10: now also U3.16 (2B3)
- net SD11: now also U3.17 (2B4)
- net SD12: now also U3.19 (2B5)
- net SD13: now also U3.20 (2B6)
- net SD14: now also U3.22 (2B7)
- net SD15: now also U3.23 (2B8)
- net SD2: now also U2.15 (D2), U3.5 (1B3)
- net SD3: now also U2.17 (D3), U3.6 (1B4)
- net SD4: now also U2.18 (D4), U3.8 (1B5)
- net SD5: now also U2.19 (D5), U3.9 (1B6)
- net SD6: now also U2.20 (D6), U3.11 (1B7)
- net SD7: now also U2.21 (D7), U3.12 (1B8)
- net SD8: now also U3.13 (2B1)
- net SD9: now also U3.14 (2B2)
- net VCC_ANA: now also C7.1, C8.1, C9.1, R3.2, U1.W6 (VCC_A)
- net VCC_CPU: now also C2.1, C4.1, C6.1, R2.2, U1.K4 (VCC_CPU), U1.L4 (VCC_CPU), U1.M4 (VCC_CPU), U1.N4 (VCC_CPU), U1.P4 (VCC_CPU), U1.R4 (VCC_CPU), U1.T4 (VCC_CPU)
- net VCC_RTC: now also U1.W7 (VCC_RTC)
- new net: U5.11 (NC), U5.15 (NC), U5.16 (NC), U5.17 (NC), U5.18 (NC), U5.33 (NC), U5.34 (NC), U5.35 (NC), U5.40 (NC)
- new net: U1.M3 (RESERVED), U1.N2 (RESERVED), U1.P1 (RESERVED), U1.P3 (RESERVED), U1.R2 (RESERVED), U1.R3 (RESERVED), U1.T2 (RESERVED), U1.U1 (RESERVED), U1.V1 (RESERVED), U1.W5 (RESERVED)
- new net: U4.11 (NC), U4.15 (NC), U4.16 (NC), U4.17 (NC), U4.18 (NC), U4.33 (NC), U4.34 (NC), U4.35 (NC), U4.40 (NC)
- new net +5V: C10.1, C12.1, U2.32 (VCC), U3.18 (VCCB), U3.7 (VCCB)
- new net D16: U1.G3 (SD0/D16), U3.47 (1A1), U5.2 (D0)
- new net D17: U1.F2 (SD1/D17), U3.46 (1A2), U5.3 (D1)
- new net D18: U1.H3 (SD2/D18), U3.44 (1A3), U5.4 (D2)
- new net D19: U1.G2 (SD3/D19), U3.43 (1A4), U5.5 (D3)
- new net D20: U1.F1 (SD4/D20), U3.41 (1A5), U5.7 (D4)
- new net D21: U1.H2 (SD5/D21), U3.40 (1A6), U5.8 (D5)
- new net D22: U1.G1 (SD6/D22), U3.38 (1A7), U5.9 (D6)
- new net D23: U1.J2 (SD7/D23), U3.37 (1A8), U5.10 (D7)
- new net D24: U1.K3 (SD8/D24), U3.36 (2A1), U5.41 (D8)
- new net D25: U1.K2 (SD9/D25), U3.35 (2A2), U5.42 (D9)
- new net D26: U1.J1 (SD10/D26), U3.33 (2A3), U5.43 (D10)
- new net D27: U1.K1 (SD11/D27), U3.32 (2A4), U5.44 (D11)
- new net D28: U1.L1 (SD12/D28), U3.30 (2A5), U5.46 (D12)
- new net D29: U1.L2 (SD13/D29), U3.29 (2A6), U5.47 (D13)
- new net D30: U1.N1 (SD14/D30), U3.27 (2A7), U5.48 (D14)
- new net D31: U1.L3 (SD15/D31), U3.26 (2A8), U5.49 (D15)
- new net MA0: U1.C10 (MA0/CFG0), U4.19 (A0), U5.19 (A0)
- new net MA1: U1.B11 (MA1/CFG1), U4.20 (A1), U5.20 (A1)
- new net MA10: U1.C13 (MA10), U4.31 (A10), U5.31 (A10)
- new net MA11: U1.A16 (MA11), U4.32 (A11), U5.32 (A11)
- new net MA2: U1.A12 (MA2), U4.21 (A2), U5.21 (A2)
- new net MA3: U1.B12 (MA3/CFG3), U4.22 (A3), U5.22 (A3)
- new net MA4: U1.C11 (MA4), U4.23 (A4), U5.23 (A4)
- new net MA5: U1.A14 (MA5), U4.24 (A5), U5.24 (A5)
- new net MA6: U1.B13 (MA6), U4.27 (A6), U5.27 (A6)
- new net MA7: U1.C12 (MA7), U4.28 (A7), U5.28 (A7)
- new net MA8: U1.A15 (MA8), U4.29 (A8), U5.29 (A8)
- new net MA9: U1.B14 (MA9), U4.30 (A9), U5.30 (A9)
- new net SA0: U1.T20 (SA0), U2.12 (A0)
- new net SA1: U1.P19 (SA1), U2.11 (A1)
- new net SA10: U1.L18 (SA10), U2.23 (A10)
- new net SA11: U1.L20 (SA11), U2.25 (A11)
- new net SA12: U1.K20 (SA12), U2.4 (A12)
- new net SA13: U1.K19 (SA13), U2.28 (A13)
- new net SA14: U1.J20 (SA14), U2.29 (A14)
- new net SA15: U1.K18 (SA15), U2.3 (A15)
- new net SA16: U1.K17 (SA16), U2.2 (A16)
- new net SA17: U1.J19 (SA17), U2.30 (A17)
- new net SA18: U1.H20 (SA18), U2.1 (A18)
- new net SA19: U1.J18 (SA19)
- new net SA2: U1.R20 (SA2), U2.10 (A2)
- new net SA20: U1.H19 (SA20)
- new net SA21: U1.G20 (SA21)
- new net SA22: U1.G19 (SA22)
- new net SA23: U1.H18 (SA23)
- new net SA24: U1.F20 (SA24)
- new net SA25: U1.H17 (SA25)
- new net SA3: U1.N18 (SA3), U2.9 (A3)
- new net SA4: U1.P20 (SA4), U2.8 (A4)
- new net SA5: U1.N19 (SA5), U2.7 (A5)
- new net SA6: U1.N20 (SA6), U2.6 (A6)
- new net SA7: U1.M18 (SA7), U2.5 (A7)
- new net SA8: U1.M20 (SA8), U2.27 (A8)
- new net SA9: U1.L19 (SA9), U2.26 (A9)
- new net ~{CASL0}: U1.B15 (~{CASL0}), U4.38 (~{LCAS})
- new net ~{CASL1}: U1.C14 (~{CASL1}), U4.37 (~{UCAS})
- new net ~{CASL2}: U1.B19 (~{CASL2}), U5.38 (~{LCAS})
- new net ~{CASL3}: U1.D16 (~{CASL3}), U5.37 (~{UCAS})
- new net ~{DBUFOE}: U1.C4 (GPIO_CS4/~{DBUFOE}), U3.25 (2~{OE}), U3.48 (1~{OE})
- new net ~{DBUFRDH}: U1.D17 (GPIO_CS3/~{DBUFRDH}), U3.24 (2DIR)
- new net ~{DBUFRDL}: U1.C18 (GPIO_CS2/~{DBUFRDL}), U3.1 (1DIR)
- new net ~{MWE}: U1.A11 (~{MWE}), U4.13 (WE), U5.13 (WE)
- new net ~{RAS0}: U1.C15 (~{RAS0}), U4.14 (~{RAS}), U5.14 (~{RAS})
- new net ~{ROMCS0}: U1.R18 (~{ROMCS0}), U2.22 (CE)
- new net ~{ROMRD}: U1.V20 (~{ROMRD}), U2.24 (OE)
- new net ~{ROMWR}: U1.U19 (~{ROMWR}), U2.31 (WE)
- no-connect marks 0 -> 8
Other:
- note added: "ISA Level Shifter"
- note added: "System ROM"
- note removed: "CPU Power Rails"

Commit message: More schematic work
Parts:
- added C15: 470p, symbol Device:C_Small
- added C16: 22p, symbol Device:C_Small
- added C17: 10n, symbol Device:C_Small
- added C18: 1n, symbol Device:C_Small
- added C19: 330p, symbol Device:C_Small
- added C20: 15p, symbol Device:C_Small
- added C21, C22: 0.1u, symbol Device:C_Small
- added R4, R5, R6: 4.7k, symbol Device:R_Small
- added Y1: 32.768kHz, symbol Device:Crystal_Small
- C13, C14: value 0.1u -> 10u
Connections:
- net +3V3: now also C21.1, C22.1
- net GND: now also U1.Y5 (GND_ANALOG), C21.2, C22.2
- net VCC_ANA: now also C15.1, C16.1, C17.1, C18.2, C19.1, C20.1
- net at U1.V5 (LF_HS): now also C20.2, R6.2
- net at U1.W4 (LF_LS): now also C16.2, R4.2
- net at U1.Y3 (LF_INT): now also C18.1, R5.2
- net at U1.Y4 (32KXTAL2): now also Y1.1
- net at U1.Y6 (32KXTAL1): now also Y1.2
- new net: C19.2, R6.1
- new net: C15.2, R4.1
- new net: C17.2, R5.1
Other:
- note added: "System RAM"
- note added: "System on Chip"
- moved on the sheet: C10, C11, C12, C13, C14, U1, U2, U3, U4, U5
